File: Kicad/N-Con-Board-2026/N-Con-Board-2026.kicad_pcb (KiCad board)
At the start: 2 copper layers, 105 x 55 mm, 22 parts, among them J1 SMA-AMP-In, J2 N-Type-Antenna, J3 Rig N-Type, J4 12v Bias Out, J5 AMP/LPF Output, J6 PTT, J7 12v Input, K1 G2RL-1-E-DC12, K2 G2RL-1-E-DC12, K3 HK4100F-DC12V-SHG, SW1 SW_Push_Test

Commit message: Update N-Con-Board
Parts:
- moved J4 2.49 mm to (114.6, 73.9)
Routing:
- net Net-(D1-K): track 77.1 -> 78.2 mm
Other:
- board text added: "N-Type Board Rev.2e"
- board text removed: "N-Type Board Rev.2d"
